File: amplifiers/pa/pa.kicad_pcb (KiCad board)
At the start: 2 copper layers, 10 parts, among them IC1 PHA-202+, J1 PWR, P1 RF IN, P2 RF OUT, X1 M3 Hole, X2 M3 Hole

Commit message: finished pcbs
Parts:
- moved L1 55.6 mm to (66.8, 82.0), turned to 270 degrees
- moved IC1 54.4 mm to (61.4, 84.9)
- moved C1 51.0 mm to (56.5, 84.3)
- moved C3 47.5 mm to (73.5, 84.3)
- moved C2 44.7 mm to (69.6, 80.0)
- moved J1 44.3 mm to (65.0, 74.0)
- moved P2 42.8 mm to (77.3, 84.3), turned to 270 degrees
- moved P1 41.5 mm to (52.7, 84.3), turned to 90 degrees
- moved X1 27.6 mm to (53.5, 73.5)
- moved X2 22.9 mm to (76.5, 73.5)
Routing:
- net GND: track 0.00 -> 20.1 mm, vias 0 -> 48
- net Net-(C3-Pad1): track 0.00 -> 14.1 mm
- net 12v: track 0.00 -> 8.70 mm
- net Net-(C3-Pad2): track 0.00 -> 3.35 mm
- net Net-(C1-Pad1): track 0.00 -> 3.35 mm
- net Net-(C1-Pad2): track 0.00 -> 1.72 mm
- added copper zone on B.Cu, net GND
- added copper zone on F.Cu, net GND
- added copper zone on F.Cu, net Net-(C3-Pad1)
Other:
- board outline added: 30 x 20 mm
- net class Default: clearance 0.2 -> 0.15; trace_width 0.25 -> 0.2
- rule pad_to_mask_clearance: 0.051 -> 0
- rule trace_clearance: 0.2 -> 0.15
- rule trace_min: 0.2 -> 0.15
- rule via_min_drill: 0.3 -> 0.4
- rule via_min_size: 0.4 -> 0.8
