File: amplifiers/pa/pa.sch (KiCad schematic (older format))
At the start: 10 parts, among them IC1 PHA-202+, J1 PWR, P1 RF IN, P2 RF OUT, X1 M3 Hole, X2 M3 Hole

Commit message: generated gerbers
Parts:
- J1: RS (none) -> 512-8585
Changed lines of the file:
@@
 EESchema Schematic File Version 4
+LIBS:pa-cache
 EELAYER 26 0
 EELAYER END
@@
 F 2 "agg:B02B-PASK" H 1525 1325 50  0001 C CNN
 F 3 "" H 1525 1325 50  0001 C CNN
+F 4 "512-8585" H 1525 1325 50  0001 C CNN "RS"
 	1    1525 1325
 	1    0    0    -1
