File: amplifiers/lna/lna.sch (KiCad schematic (older format))
At the start: 14 parts, among them IC1 CMA-83LN+, J1 MICROUSB, P1 RF IN, P2 RF OUT, X1 M3 Hole, X2 M3 Hole, X3 M3 Hole, X4 M3 Hole

Commit message: finsihed amplifier schematics
Parts:
- removed IC1: CMA-83LN+, agg:DL1721, symbol agg-kicad:CMA-83LN+
- removed X3, X4: M3 Hole, agg:M3_MOUNT, symbol agg-kicad:PART
- added IC1: PMA3-83LN+, agg:DQ1225, symbol agg-kicad:PMA3-83LN+
Connections:
- wire segments 42 -> 51
Other:
- moved on the sheet: C1, C2

Commit message: generated gerbers
Parts:
- J1: Farnell 1568023 -> (none); RS (none) -> 702-5488
Changed lines of the file:
@@
 F 2 "agg:MICROUSB_MOLEX_47589-0001" H 1350 950 50  0001 L CNN
 F 3 "" H 1800 1650 50  0001 C CNN
-F 4 "1568023" H 1350 850 50  0001 L CNN "Farnell"
+F 4 "702-5488" H 1350 850 50  0001 L CNN "RS"
 	1    1500 1450
 	1    0    0    -1
